File: CAD/Control shield/control.brd (EAGLE design)
At the start: 41.5 x 35.4 mm, 7 parts

Commit message: Added another 3-pin header for CAN to make debugging easier.
Parts:
- added JP3: (no value), ASL:1X03_LOCK
- R1, R2: value (none) -> 330
- moved JP1 16.5 mm to (31.0, 23.1), turned to 180 degrees
- moved JP2 2.88 mm to (37.7, 13.3)
Connections:
- new net CAN_HI: JP3.1, U$1.P$25
- new net CAN_LO: JP3.2, U$1.P$26
- new net GND3: JP3.3, U$1.P$28
- net GND: now also U$1.P$16; no longer U$1.P$28
- net UART2_RX: now also U$1.P$18; no longer U$1.P$22
- net UART2_TX: now also U$1.P$22; no longer U$1.P$18
Routing:
- net GND3: track 0.00 -> 22.6 mm
- net CAN_LO: track 0.00 -> 19.6 mm
- net CAN_HI: track 0.00 -> 19.5 mm
- net VOLTAGE_SENSE: track 10.3 -> 7.37 mm
- net UART2_RX: track 7.49 -> 9.33 mm
- net CURRENT_SENSE: track 9.53 -> 8.16 mm
- net GND: track 7.24 -> 8.53 mm
Other:
- board text added: "CAN"
- board text added: "CANHI"
- board text added: "CANLO"
- board text added: "UART2 HIL/REVO_GS"
- board text removed: "HIL REVO_GS"
Changed lines of the file:
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@@
 <setting verticaltext="up"/>
 </settings>
-<grid distance="0.01" unitdist="inch" unit="inch" style="lines" multiple="1" display="no" altdistance="0.025" altunitdist="inch" altunit="inch"/>
+<grid distance="0.005" unitdist="inch" unit="inch" style="lines" multiple="1" display="no" altdistance="0.025" altunitdist="inch" altunit="inch"/>
 <layers>
 <layer number="1" name="Top" color="4" fill="1" visible="yes" active="yes"/>
@@
 <board>
 <plain>
-<text x="13.716" y="22.352" size="1.778" layer="21" font="vector" ratio="12" rot="R270">GND</text>
-<text x="21.336" y="22.352" size="1.778" layer="21" font="vector" ratio="12" rot="R270">RX</text>
-<text x="23.622" y="22.352" size="1.778" layer="21" font="vector" ratio="12" rot="R270">TX</text>
-<text x="34.036" y="16.256" size="1.778" layer="21" font="vector" ratio="12" rot="R180">C_SENSE</text>
-<text x="34.036" y="13.716" size="1.778" layer="21" font="vector" ratio="12" rot="R180">V_SENSE</text>
+<text x="30.226" y="21.59" size="1.778" layer="21" font="vector" ratio="12" rot="R270">GND</text>
+<text x="22.606" y="21.59" size="1.778" layer="21" font="vector" ratio="12" rot="R270">RX</text>
+<text x="19.812" y="21.59" size="1.778" layer="21" font="vector" ratio="12" rot="R270">TX</text>
+<text x="36.068" y="14.224" size="1.778" layer="21" font="vector" ratio="12" rot="R180">C_SENSE</text>
+<text x="36.068" y="11.684" size="1.778" layer="21" font="vector" ratio="12" rot="R180">V_SENSE</text>
 <text x="35.052" y="31.75" size="1.778" layer="21" font="vector" ratio="12">AUTOMODE</text>
-<text x="34.544" y="24.638" size="1.778" layer="21" font="vector" ratio="12">GPS</text>
-<text x="9.652" y="25.654" size="1.778" layer="21" font="vector" ratio="12">HIL
-REVO_GS</text>
+<text x="35.052" y="24.892" size="1.778" layer="21" font="vector" ratio="12">GPS</text>
+<text x="16.129" y="24.892" size="1.778" layer="21" font="vector" ratio="12">UART2
+HIL/REVO_GS</text>
+<text x="13.843" y="15.24" size="1.778" layer="21" font="vector" ratio="12">CANHI</text>
+<text x="13.843" y="10.16" size="1.778" layer="21" font="vector" ratio="12">GND</text>
+<text x="13.843" y="12.7" size="1.778" layer="21" font="vector" ratio="12">CANLO</text>
+<text x="10.033" y="17.78" size="1.778" layer="21" font="vector" ratio="12">CAN</text>
 </plain>
 <attributes>
@@
 <elements>
 <element name="U$1" library="ASL" package="CAN_NODE_SHIELD" value="CAN_NODE_SHIELD" x="0" y="0"/>
-<element name="JP1" library="ASL" package="1X06-SIP_LOCK" value="" x="14.478" y="23.876" smashed="yes">
-<attribute name="NAME" x="25.654" y="25.4" size="1.143" layer="25" font="vector" ratio="14"/>
-<attribute name="VALUE" x="13.208" y="20.955" size="1.27" layer="27" font="vector"/>
+<element name="JP1" library="ASL" package="1X06-SIP_LOCK" value="" x="30.988" y="23.114" smashed="yes" rot="R180">
+<attribute name="NAME" x="16.891" y="23.622" size="1.143" layer="25" font="vector" ratio="14" rot="R180"/>
+<attribute name="VALUE" x="32.258" y="26.035" size="1.27" layer="27" font="vector" rot="R180"/>
 </element>
 <element name="LED1" library="ASL" package="LED-1206" value="" x="37.338" y="23.368" smashed="yes">
 <attribute name="NAME" x="39.497" y="21.971" size="1.143" layer="25" font="vector" ratio="14" rot="R180"/>
 <attribute name="VALUE" x="36.322" y="21.59" size="0.4064" layer="27"/>
+<attribute name="COLOR" value="green" x="37.338" y="23.368" size="1.778" layer="27" display="off"/>
 </element>
 <element name="LED2" library="ASL" package="LED-1206" value="" x="37.338" y="30.226" smashed="yes">
 <attribute name="NAME" x="39.497" y="28.829" size="1.143" layer="25" font="vector" ratio="14" rot="R180"/>
 <attribute name="VALUE" x="36.322" y="28.448" size="0.4064" layer="27"/>
-</element>
-<element name="R1" library="ASL" package="0805" value="" x="41.402" y="21.082" smashed="yes">
-<attribute name="NAME" x="42.672" y="20.2565" size="1.143" layer="25" font="vector" ratio="14" rot="R180"/>
-<attribute name="VALUE" x="40.386" y="19.685" size="0.4064" layer="27"/>
-</element>
-<element name="R2" library="ASL" package="0805" value="" x="32.766" y="32.766" smashed="yes" rot="R90">
+<attribute name="COLOR" value="amber" x="37.338" y="30.226" size="1.778" layer="27" display="off"/>
+</element>
+<element name="R1" library="ASL" package="0805" value="330" x="41.402" y="21.082" smashed="yes">
+<attribute name="NAME" x="42.672" y="20.1295" size="1.143" layer="25" font="vector" ratio="14" rot="R180"/>
+</element>
+<element name="R2" library="ASL" package="0805" value="330" x="32.766" y="32.766" smashed="yes" rot="R90">
 <attribute name="NAME" x="33.782" y="31.1785" size="1.143" layer="25" font="vector" ratio="14" rot="R180"/>
-<attribute name="VALUE" x="34.163" y="31.75" size="0.4064" layer="27" rot="R90"/>
-</element>
-<element name="JP2" library="ASL" package="1X03_LOCK" value="" x="35.56" y="15.24" smashed="yes" rot="R270">
-<attribute name="NAME" x="33.9598" y="16.8148" size="1.143" layer="25" font="vector" ratio="14"/>
+</element>
+<element name="JP2" library="ASL" package="1X03_LOCK" value="" x="37.719" y="13.335" smashed="yes" rot="R270">
+<attribute name="NAME" x="36.1188" y="14.9098" size="1.143" layer="25" font="vector" ratio="14"/>
+</element>
+<element name="JP3" library="ASL" package="1X03_LOCK" value="" x="12.192" y="16.129" smashed="yes" rot="R270">
+<attribute name="NAME" x="13.6652" y="9.3472" size="1.27" layer="25" ratio="15" rot="R180"/>
 </element>
 </elements>
@@
 <contactref element="U$1" pad="P$8"/>
 <contactref element="JP2" pad="1"/>
-<wire x1="35.687" y1="15.24" x2="36.322" y2="15.875" width="0.762" layer="16"/>
-<wire x1="36.322" y1="15.875" x2="44.958" y2="15.875" width="0.762" layer="16"/>
+<wire x1="37.846" y1="13.335" x2="42.418" y2="13.335" width="0.762" layer="16"/>
+<wire x1="42.418" y1="13.335" x2="44.958" y2="15.875" width="0.762" layer="16"/>
 </signal>
 <signal name="VOLTAGE_SENSE">
 <contactref element="U$1" pad="P$4"/>
 <contactref element="JP2" pad="2"/>
-<wire x1="35.433" y1="12.7" x2="37.338" y2="10.795" width="0.762" layer="16"/>
-<wire x1="37.338" y1="10.795" x2="44.958" y2="10.795" width="0.762" layer="16"/>
+<wire x1="44.958" y1="10.795" x2="37.592" y2="10.795" width="0.762" layer="16"/>
 </signal>
 <signal name="UART2_RX">
+<contactref element="JP1" pad="4"/>
+<contactref element="U$1" pad="P$18"/>
+<wire x1="27.178" y1="31.115" x2="27.178" y2="27.178" width="0.762" layer="16"/>
+<wire x1="27.178" y1="27.178" x2="23.368" y2="23.368" width="0.762" layer="16"/>
+</signal>
+<signal name="UART2_TX">
+<contactref element="JP1" pad="5"/>
 <contactref element="U$1" pad="P$22"/>
-<contactref element="JP1" pad="4"/>
-<wire x1="22.098" y1="23.622" x2="22.098" y2="31.115" width="0.762" layer="16"/>
-</signal>
-<signal name="UART2_TX">
-<contactref element="U$1" pad="P$18"/>
-<contactref element="JP1" pad="5"/>
-<wire x1="24.638" y1="23.876" x2="27.178" y2="26.416" width="0.762" layer="16"/>
-<wire x1="27.178" y1="26.416" x2="27.178" y2="31.115" width="0.762" layer="16"/>
+<wire x1="22.098" y1="31.115" x2="20.828" y2="29.845" width="0.762" layer="16"/>
+<wire x1="20.828" y1="23.114" x2="20.828" y2="29.845" width="0.762" layer="16"/>
 </signal>
 <signal name="GND" class="1">
 <contactref element="JP1" pad="1"/>
-<contactref element="U$1" pad="P$28"/>
-<wire x1="14.478" y1="23.876" x2="14.478" y2="31.115" width="0.762" layer="16"/>
+<contactref element="U$1" pad="P$16"/>
+<wire x1="29.718" y1="31.115" x2="30.988" y2="29.845" width="0.762" layer="16"/>
+<wire x1="30.988" y1="29.845" x2="30.988" y2="23.114" width="0.762" layer="16"/>
 </signal>
 <signal name="LED_AUTOMODE">
@@
 <wire x1="38.838" y1="24.027" x2="39.37" y2="23.495" width="0.762" layer="1"/>
 </signal>
+<signal name="GND3">
+<contactref element="JP3" pad="3"/>
+<contactref element="U$1" pad="P$28"/>
+<wire x1="14.478" y1="31.115" x2="10.287" y2="26.924" width="0.762" layer="16"/>
+<wire x1="10.287" y1="26.924" x2="10.287" y2="13.081" width="0.762" layer="16"/>
+<wire x1="10.287" y1="13.081" x2="12.319" y2="11.049" width="0.762" layer="16"/>
+</signal>
+<signal name="CAN_LO">
+<contactref element="JP3" pad="2"/>
+<contactref element="U$1" pad="P$26"/>
+<wire x1="12.065" y1="13.589" x2="15.748" y2="17.272" width="0.762" layer="16"/>
+<wire x1="15.748" y1="17.272" x2="15.748" y2="24.13" width="0.762" layer="16"/>
+<wire x1="15.748" y1="24.13" x2="17.018" y2="25.4" width="0.762" layer="16"/>
+<wire x1="17.018" y1="25.4" x2="17.018" y2="31.115" width="0.762" layer="16"/>
+</signal>
+<signal name="CAN_HI" class="2">
+<contactref element="JP3" pad="1"/>
+<contactref element="U$1" pad="P$25"/>
+<wire x1="12.319" y1="16.129" x2="14.224" y2="18.034" width="0.254" layer="16"/>
+<wire x1="14.224" y1="18.034" x2="14.224" y2="26.162" width="0.254" layer="16"/>
+<wire x1="14.224" y1="26.162" x2="15.748" y2="27.686" width="0.254" layer="16"/>
+<wire x1="15.748" y1="27.686" x2="15.748" y2="32.385" width="0.254" layer="16"/>
+<wire x1="15.748" y1="32.385" x2="17.018" y2="33.655" width="0.254" layer="16"/>
+</signal>
 </signals>

Commit message: Updated the control and rudder shields to be single-sided on the top for a board run. Also updated their documentation.
Changed lines of the file:
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@@
 <contactref element="U$1" pad="P$8"/>
 <contactref element="JP2" pad="1"/>
-<wire x1="37.846" y1="13.335" x2="42.418" y2="13.335" width="0.762" layer="16"/>
-<wire x1="42.418" y1="13.335" x2="44.958" y2="15.875" width="0.762" layer="16"/>
+<wire x1="37.846" y1="13.335" x2="42.418" y2="13.335" width="0.762" layer="1"/>
+<wire x1="42.418" y1="13.335" x2="44.958" y2="15.875" width="0.762" layer="1"/>
 </signal>
 <signal name="VOLTAGE_SENSE">
 <contactref element="U$1" pad="P$4"/>
 <contactref element="JP2" pad="2"/>
-<wire x1="44.958" y1="10.795" x2="37.592" y2="10.795" width="0.762" layer="16"/>
+<wire x1="44.958" y1="10.795" x2="37.592" y2="10.795" width="0.762" layer="1"/>
 </signal>
 <signal name="UART2_RX">
 <contactref element="JP1" pad="4"/>
 <contactref element="U$1" pad="P$18"/>
-<wire x1="27.178" y1="31.115" x2="27.178" y2="27.178" width="0.762" layer="16"/>
-<wire x1="27.178" y1="27.178" x2="23.368" y2="23.368" width="0.762" layer="16"/>
+<wire x1="27.178" y1="31.115" x2="27.178" y2="27.178" width="0.762" layer="1"/>
+<wire x1="27.178" y1="27.178" x2="23.368" y2="23.368" width="0.762" layer="1"/>
 </signal>
 <signal name="UART2_TX">
 <contactref element="JP1" pad="5"/>
 <contactref element="U$1" pad="P$22"/>
-<wire x1="22.098" y1="31.115" x2="20.828" y2="29.845" width="0.762" layer="16"/>
-<wire x1="20.828" y1="23.114" x2="20.828" y2="29.845" width="0.762" layer="16"/>
+<wire x1="22.098" y1="31.115" x2="20.828" y2="29.845" width="0.762" layer="1"/>
+<wire x1="20.828" y1="23.114" x2="20.828" y2="29.845" width="0.762" layer="1"/>
 </signal>
 <signal name="GND" class="1">
 <contactref element="JP1" pad="1"/>
 <contactref element="U$1" pad="P$16"/>
-<wire x1="29.718" y1="31.115" x2="30.988" y2="29.845" width="0.762" layer="16"/>
-<wire x1="30.988" y1="29.845" x2="30.988" y2="23.114" width="0.762" layer="16"/>
+<wire x1="29.718" y1="31.115" x2="30.988" y2="29.845" width="0.762" layer="1"/>
+<wire x1="30.988" y1="29.845" x2="30.988" y2="23.114" width="0.762" layer="1"/>
 </signal>
 <signal name="LED_AUTOMODE">
@@
 <contactref element="JP3" pad="3"/>
 <contactref element="U$1" pad="P$28"/>
-<wire x1="14.478" y1="31.115" x2="10.287" y2="26.924" width="0.762" layer="16"/>
-<wire x1="10.287" y1="26.924" x2="10.287" y2="13.081" width="0.762" layer="16"/>
-<wire x1="10.287" y1="13.081" x2="12.319" y2="11.049" width="0.762" layer="16"/>
+<wire x1="14.478" y1="31.115" x2="10.287" y2="26.924" width="0.762" layer="1"/>
+<wire x1="10.287" y1="26.924" x2="10.287" y2="13.081" width="0.762" layer="1"/>
+<wire x1="10.287" y1="13.081" x2="12.319" y2="11.049" width="0.762" layer="1"/>
 </signal>
 <signal name="CAN_LO">
 <contactref element="JP3" pad="2"/>
 <contactref element="U$1" pad="P$26"/>
-<wire x1="12.065" y1="13.589" x2="15.748" y2="17.272" width="0.762" layer="16"/>
-<wire x1="15.748" y1="17.272" x2="15.748" y2="24.13" width="0.762" layer="16"/>
-<wire x1="15.748" y1="24.13" x2="17.018" y2="25.4" width="0.762" layer="16"/>
-<wire x1="17.018" y1="25.4" x2="17.018" y2="31.115" width="0.762" layer="16"/>
+<wire x1="12.065" y1="13.589" x2="15.748" y2="17.272" width="0.762" layer="1"/>
+<wire x1="15.748" y1="17.272" x2="15.748" y2="24.13" width="0.762" layer="1"/>
+<wire x1="15.748" y1="24.13" x2="17.018" y2="25.4" width="0.762" layer="1"/>
+<wire x1="17.018" y1="25.4" x2="17.018" y2="31.115" width="0.762" layer="1"/>
 </signal>
 <signal name="CAN_HI" class="2">
 <contactref element="JP3" pad="1"/>
 <contactref element="U$1" pad="P$25"/>
-<wire x1="12.319" y1="16.129" x2="14.224" y2="18.034" width="0.254" layer="16"/>
-<wire x1="14.224" y1="18.034" x2="14.224" y2="26.162" width="0.254" layer="16"/>
-<wire x1="14.224" y1="26.162" x2="15.748" y2="27.686" width="0.254" layer="16"/>
-<wire x1="15.748" y1="27.686" x2="15.748" y2="32.385" width="0.254" layer="16"/>
-<wire x1="15.748" y1="32.385" x2="17.018" y2="33.655" width="0.254" layer="16"/>
+<wire x1="12.319" y1="16.129" x2="14.224" y2="18.034" width="0.254" layer="1"/>
+<wire x1="14.224" y1="18.034" x2="14.224" y2="26.162" width="0.254" layer="1"/>
+<wire x1="14.224" y1="26.162" x2="15.748" y2="27.686" width="0.254" layer="1"/>
+<wire x1="15.748" y1="27.686" x2="15.748" y2="32.385" width="0.254" layer="1"/>
+<wire x1="15.748" y1="32.385" x2="17.018" y2="33.655" width="0.254" layer="1"/>
 </signal>
 </signals>

Commit message: Primary node shield:  * Removed defunct HIL/Revolution GS UART connection
Parts:
- removed JP1: (no value), ASL:1X06-SIP_LOCK
Connections:
- removed net UART2_RX: JP1.4, U$1.P$18
- removed net UART2_TX: JP1.5, U$1.P$22
- net GND: no longer JP1.1
Routing:
- net UART2_RX: track 9.33 -> 0.00 mm
- net UART2_TX: track 8.53 -> 0.00 mm
- net GND: track 8.53 -> 0.00 mm
Other:
- board text removed: "RX"
- board text removed: "TX"
- board text removed: "UART2 HIL/REVO_GS"
Changed lines of the file:
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@@
 <board>
 <plain>
-<text x="30.226" y="21.59" size="1.778" layer="21" font="vector" ratio="12" rot="R270">GND</text>
-<text x="22.606" y="21.59" size="1.778" layer="21" font="vector" ratio="12" rot="R270">RX</text>
-<text x="19.812" y="21.59" size="1.778" layer="21" font="vector" ratio="12" rot="R270">TX</text>
 <text x="36.068" y="14.224" size="1.778" layer="21" font="vector" ratio="12" rot="R180">C_SENSE</text>
 <text x="36.068" y="11.684" size="1.778" layer="21" font="vector" ratio="12" rot="R180">V_SENSE</text>
 <text x="35.052" y="31.75" size="1.778" layer="21" font="vector" ratio="12">AUTOMODE</text>
 <text x="35.052" y="24.892" size="1.778" layer="21" font="vector" ratio="12">GPS</text>
-<text x="16.129" y="24.892" size="1.778" layer="21" font="vector" ratio="12">UART2
-HIL/REVO_GS</text>
 <text x="13.843" y="15.24" size="1.778" layer="21" font="vector" ratio="12">CANHI</text>
 <text x="13.843" y="10.16" size="1.778" layer="21" font="vector" ratio="12">GND</text>
@@
 <elements>
 <element name="U$1" library="ASL" package="CAN_NODE_SHIELD" value="CAN_NODE_SHIELD" x="0" y="0"/>
-<element name="JP1" library="ASL" package="1X06-SIP_LOCK" value="" x="30.988" y="23.114" smashed="yes" rot="R180">
-<attribute name="NAME" x="16.891" y="23.622" size="1.143" layer="25" font="vector" ratio="14" rot="R180"/>
-<attribute name="VALUE" x="32.258" y="26.035" size="1.27" layer="27" font="vector" rot="R180"/>
-</element>
 <element name="LED1" library="ASL" package="LED-1206" value="" x="37.338" y="23.368" smashed="yes">
 <attribute name="NAME" x="39.497" y="21.971" size="1.143" layer="25" font="vector" ratio="14" rot="R180"/>
@@
 <wire x1="44.958" y1="10.795" x2="37.592" y2="10.795" width="0.762" layer="1"/>
 </signal>
-<signal name="UART2_RX">
-<contactref element="JP1" pad="4"/>
-<contactref element="U$1" pad="P$18"/>
-<wire x1="27.178" y1="31.115" x2="27.178" y2="27.178" width="0.762" layer="1"/>
-<wire x1="27.178" y1="27.178" x2="23.368" y2="23.368" width="0.762" layer="1"/>
-</signal>
-<signal name="UART2_TX">
-<contactref element="JP1" pad="5"/>
-<contactref element="U$1" pad="P$22"/>
-<wire x1="22.098" y1="31.115" x2="20.828" y2="29.845" width="0.762" layer="1"/>
-<wire x1="20.828" y1="23.114" x2="20.828" y2="29.845" width="0.762" layer="1"/>
-</signal>
 <signal name="GND" class="1">
-<contactref element="JP1" pad="1"/>
 <contactref element="U$1" pad="P$16"/>
-<wire x1="29.718" y1="31.115" x2="30.988" y2="29.845" width="0.762" layer="1"/>
-<wire x1="30.988" y1="29.845" x2="30.988" y2="23.114" width="0.762" layer="1"/>
 </signal>
 <signal name="LED_AUTOMODE">
@@
 </board>
 </drawing>
-<compatibility>
-<note version="6.3" minversion="6.2.2" severity="warning">
-Since Version 6.2.2 text objects can contain more than one line,
-which will not be processed correctly with this version.
-</note>
-</compatibility>
 </eagle>
